Commit message: polecart task working

File: urdf/cartpole_v0.urdf (robot description, URDF)
Before this commit: robot cartpole_v0, 4 links, 3 joints
Links:
- link bar_link: geometry visual box size=0.05 0.05 0.8
Joints:
- joint cartpole_joint: limit lower=-1.57 upper=1.57 effort=1 velocity=100 -> lower=-6.28 upper=6.28 effort=0 velocity=1000; origin xyz=0 0 0.32 rpy=0 0 0 -> xyz=0 -0.2 0.32 rpy=0 0 0
